Commit message: running arm model without tuning

File: components/urdf/wam/arm.urdf.xacro (robot description, xacro)
@@ -24,6 +24,6 @@
 -->
 <robot xmlns:xacro="http://www.ros.org/wiki/xacro">
-    <xacro:include filename="$(find waterloo_steel_description)/urdf/wam/common.urdf.xacro"/>
-    <xacro:include filename="$(find waterloo_steel_description)/urdf/wam/components.urdf.xacro"/>
+    <xacro:include filename="$(find uwarl-mujoco-summit-wam-sim)/components/urdf/wam/common.urdf.xacro"/>
+    <xacro:include filename="$(find uwarl-mujoco-summit-wam-sim)/components/urdf/wam/components_V1.urdf.xacro"/>
     <xacro:macro name="wam_7dof" params="prefix parent_link xyz rpy torque_sensor">
         <xacro:arg name="torque_sensor" default="false"/>

File: components/urdf/wam/ball.urdf.xacro (robot description, xacro)
@@ -1,4 +1,4 @@
 <robot xmlns:xacro="http://www.ros.org/wiki/xacro">
-    <xacro:include filename="$(find waterloo_steel_description)/urdf/wam/common.urdf.xacro"/>
+    <xacro:include filename="$(find uwarl-mujoco-summit-wam-sim)/components/urdf/wam/common.urdf.xacro"/>
     <!-- High-leveel hand macro -->
     <xacro:macro name="bball" params="parent_link prefix xyz rpy">

File: components/urdf/wam/common.urdf.xacro (robot description, xacro)
@@ -25,5 +25,5 @@
 <robot xmlns:xacro="http://ros.org/wiki/xacro">
     <!-- Directories -->
-    <xacro:property name="models_path" value="package://waterloo_steel_description" />
+    <xacro:property name="models_path" value="package://uwarl-mujoco-summit-wam-sim/components" />
     <!-- <xacro:property name="highResModelDirectory" value="${models_path}/meshes/splitModels" /> -->
     <!-- Constants -->

File: components/urdf/wam/components.urdf.xacro (robot description, xacro)
@@ -24,6 +24,6 @@
 -->
 <robot xmlns:xacro="http://ros.org/wiki/xacro">
-    <xacro:include filename="$(find waterloo_steel_description)/urdf/wam/hand.urdf.xacro"/>
-    <xacro:include filename="$(find waterloo_steel_description)/urdf/wam/common.urdf.xacro"/>
+    <xacro:include filename="$(find uwarl-mujoco-summit-wam-sim)/components/urdf/wam/hand.urdf.xacro"/>
+    <xacro:include filename="$(find uwarl-mujoco-summit-wam-sim)/components/urdf/wam/common.urdf.xacro"/>
     <xacro:property name="b" value="0.5"/>
     <xacro:property name="M_PI" value="3.1415926535897931"/>

File: components/urdf/wam/components_V1.urdf.xacro (robot description, xacro)
@@ -24,6 +24,6 @@
 -->
 <robot xmlns:xacro="http://ros.org/wiki/xacro">
-    <xacro:include filename="$(find waterloo_steel_description)/urdf/wam/hand.urdf.xacro"/>
-    <xacro:include filename="$(find waterloo_steel_description)/urdf/wam/common.urdf.xacro"/>
+    <xacro:include filename="$(find uwarl-mujoco-summit-wam-sim)/components/urdf/wam/hand.urdf.xacro"/>
+    <xacro:include filename="$(find uwarl-mujoco-summit-wam-sim)/components/urdf/wam/common.urdf.xacro"/>
     <xacro:property name="b" value="0.5"/>
     <xacro:property name="M_PI" value="3.1415926535897931"/>
@@ -63,13 +63,13 @@
     </xacro:macro>
     <xacro:macro name="wam_shoulder_yaw" params="prefix">
-        <joint name="${prefix}/base_yaw_joint" type="revolute">
+        <joint name="${prefix}/J1" type="revolute">
             <parent link="${prefix}/base_link"/>
             <child link="${prefix}/shoulder_yaw_link"/>
             <origin xyz="0 0 0.346" rpy="0 0 0"/>
             <axis xyz="0 0 1"/>
-            <limit effort="${60*4}" lower="${-148.97 * M_PI / 180.0}" upper="${148.97 * M_PI / 180.0}" velocity="2.0"/>
+            <limit effort="${60}" lower="${-148.97 * M_PI / 180.0}" upper="${148.97 * M_PI / 180.0}" velocity="2.0"/>
             <dynamics damping="${1.8*b}" friction="0"/>
         </joint>
-        <gazebo reference="${prefix}/base_yaw_joint">
+        <gazebo reference="${prefix}/J1">
             <xacro:gz_joint/>
         </gazebo>
@@ -86,5 +86,5 @@
             <inertial>
                 <origin xyz="-.00443422 -.00066489 -0.1289039 " />
-                <mass value="${5*0.1}" /> <!-- Before, it was 10.76768767, now it is 5 from the Barett WAM spec pdf in the Mujoco simulator repo -->
+                <mass value="${5}" /> <!-- Before, it was 10.76768767, now it is 5 from the Barett WAM spec pdf in the Mujoco simulator repo -->
                 <inertia
                     ixx=".13488033"     ixy="-0.00012485"   ixz="0.00213041"
@@ -110,13 +110,13 @@
     </xacro:macro>
     <xacro:macro name="wam_shoulder_pitch" params="prefix">
-        <joint name="${prefix}/shoulder_pitch_joint" type="revolute">
+        <joint name="${prefix}/J2" type="revolute">
             <parent link="${prefix}/shoulder_yaw_link"/>
             <child link="${prefix}/shoulder_pitch_link"/>
             <origin xyz="0 0 0" rpy="${-PI/2} 0 0"/>
             <axis xyz="0 0 1"/>
-            <limit effort="${60*4}" lower="${-113.732 * M_PI / 180.0}" upper="${113.732 * M_PI / 180.0}" velocity="2.0"/>
+            <limit effort="${60}" lower="${-113.732 * M_PI / 180.0}" upper="${113.732 * M_PI / 180.0}" velocity="2.0"/>
             <dynamics damping="${0.5*b}" friction="0"/>
         </joint>
-        <gazebo reference="${prefix}/shoulder_pitch_joint">
+        <gazebo reference="${prefix}/J2">
             <xacro:gz_joint/>
         </gazebo>
@@ -141,5 +141,5 @@
             <inertial>
                 <origin xyz="-.00236981 -.01542114 .03105614 " />
-                <mass value="${3.87493756*0.1}" />
+                <mass value="${3.87493756}" />
                 <inertia
                     ixx="0.02140958"    ixy="-0.00002461"   ixz="0.00027172"
@@ -155,13 +155,13 @@
     </xacro:macro>
     <xacro:macro name="wam_upper_arm" params="prefix">
-        <joint name="${prefix}/shoulder_yaw_joint" type="revolute">
+        <joint name="${prefix}/J3" type="revolute">
             <parent link="${prefix}/shoulder_pitch_link"/>
             <child link="${prefix}/upper_arm_link"/>
             <origin xyz="0 0 0" rpy="${PI/2} 0 0"/>
             <axis xyz="0 0 1"/>
-            <limit effort="${45*4}" lower="${-160.428 * M_PI / 180.0}" upper="${160.428 * M_PI / 180.0}" velocity="2.0"/>
+            <limit effort="${45}" lower="${-160.428 * M_PI / 180.0}" upper="${160.428 * M_PI / 180.0}" velocity="2.0"/>
             <dynamics damping="${1.5*b}" friction="0"/>
         </joint>
-        <gazebo reference="${prefix}/shoulder_yaw_joint">
+        <gazebo reference="${prefix}/J3">
             <xacro:gz_joint/>
         </gazebo>
@@ -178,5 +178,5 @@
             <inertial>
                 <origin xyz="0.00683258580000000 0.000033090000000 0.392492300000000" />
-                <mass value="${2.20228141*0.1}" />
+                <mass value="${2.20228141}" />
                 <inertia
                     ixx=".05911077"     ixy="-0.00000738"   ixz="-0.00249612"
@@ -202,13 +202,13 @@
     <!-- Forearm macros -->
     <xacro:macro name="wam_forearm" params="prefix">
-        <joint name="${prefix}/elbow_pitch_joint" type="revolute">
+        <joint name="${prefix}/J4" type="revolute">
             <parent link="${prefix}/upper_arm_link"/>
             <child link="${prefix}/forearm_link"/>
             <origin xyz="0.045 0 0.55" rpy="${-PI/2} 0 0"/>
             <axis xyz="0 0 1"/>
-            <limit effort="${30*4}" lower="${-51.567 * M_PI / 180.0}" upper="${180 * M_PI / 180.0}" velocity="2.00"/>
+            <limit effort="${30}" lower="${-51.567 * M_PI / 180.0}" upper="${180 * M_PI / 180.0}" velocity="2.00"/>
             <dynamics damping="${0.8*b}" friction="0"/>
         </joint>
-        <gazebo reference="${prefix}/elbow_pitch_joint">
+        <gazebo reference="${prefix}/J4">
             <xacro:gz_joint/>
         </gazebo>
@@ -224,5 +224,5 @@
         <link name="${prefix}/forearm_link" >
             <inertial>
-                <mass value="${0.50016804*0.1}" />
+                <mass value="${0.50016804}" />
                 <origin xyz="-0.04001488 -.14271662 -.00022942 " rpy="0 0 0" />
                 <inertia
@@ -263,13 +263,13 @@
     </xacro:macro>
     <xacro:macro name="wam_wrist_yaw" params="prefix">
-        <joint name="${prefix}/wrist_yaw_joint" type="revolute">
+        <joint name="${prefix}/J5" type="revolute">
             <parent link="${prefix}/forearm_link"/>
             <child link="${prefix}/wrist_yaw_link"/>
             <origin xyz="-0.045 -0.3 0" rpy="${PI/2} 0 0"/>
             <axis xyz="0 0 1"/>
-            <limit effort="${10*2}" lower="${-260.696 * M_PI / 180.0}" upper="${71.62 * M_PI / 180.0}" velocity="2.0"/>
+            <limit effort="${10}" lower="${-260.696 * M_PI / 180.0}" upper="${71.62 * M_PI / 180.0}" velocity="2.0"/>
             <dynamics damping="${0.5*b}" friction="0"/>
         </joint>
-        <gazebo reference="${prefix}/wrist_yaw_joint">
+        <gazebo reference="${prefix}/J5">
             <xacro:gz_joint/>
         </gazebo>
@@ -286,5 +286,5 @@
             <inertial>
                 <origin xyz="0.00008921 0.00435824 -0.00511217 " />
-                <mass value="${1.05376019*0.1}" />
+                <mass value="${1.05376019}" />
                 <inertia  ixx="0.00005029" ixy="0.00000020"  ixz="0.00007582"
                     iyy="0.00007582"  iyz="-0.00000359"
@@ -310,13 +310,13 @@
     </xacro:macro>
     <xacro:macro name="wam_wrist_pitch" params="prefix">
-        <joint name="${prefix}/wrist_pitch_joint" type="revolute">
+        <joint name="${prefix}/J6" type="revolute">
             <parent link="${prefix}/wrist_yaw_link"/>
             <child link="${prefix}/wrist_pitch_link"/>
             <origin xyz="0 0 0" rpy="${-PI/2} 0 0"/>
             <axis xyz="0 0 1"/>
-            <limit effort="${10*2}" lower="${-90 * M_PI / 180.0}" upper="${90 * M_PI / 180.0}" velocity="2.00"/>
+            <limit effort="${10}" lower="${-90 * M_PI / 180.0}" upper="${90 * M_PI / 180.0}" velocity="2.00"/>
             <dynamics damping="${0.1*b}" friction="0"/>
         </joint>
-        <gazebo reference="${prefix}/wrist_pitch_joint">
+        <gazebo reference="${prefix}/J6">
             <xacro:gz_joint/>
         </gazebo>
@@ -333,5 +333,5 @@
             <inertial>
                 <origin xyz="-0.00012262 -0.02468336 -0.01703194 " rpy="0 0 0" />
-                <mass value="${0.51797364*0.1}" />
+                <mass value="${0.51797364}" />
                 <inertia
                     ixx="0.00055516"  ixy="0.00000061"  ixz="-0.00000074"
@@ -358,14 +358,14 @@
     <!-- Palm without force-torque sensor -->
     <xacro:macro name="wam_palm" params="prefix">
-        <joint name="${prefix}/palm_yaw_joint" type="revolute">
+        <joint name="${prefix}/J7" type="revolute">
             <parent link="${prefix}/wrist_pitch_link"/>
             <child link="${prefix}/wrist_palm_link"/>
             <origin xyz="0 0 0" rpy="${PI/2} 0 0"/>
             <axis xyz="0 0 1"/>
-            <limit effort="${10*2}" lower="${-171.89 * M_PI / 180.0}" upper="${171.89 * M_PI / 180.0}" velocity="2.00"/>
+            <limit effort="${10}" lower="${-171.89 * M_PI / 180.0}" upper="${171.89 * M_PI / 180.0}" velocity="2.00"/>
             <!-- 2.95 is a limit taken in from 3 due to saftey and differences between arms. -->
             <dynamics damping="${0.1*b}" friction="0"/>
         </joint>
-        <gazebo reference="${prefix}/palm_yaw_joint">
+        <gazebo reference="${prefix}/J7">
             <xacro:gz_joint/>
         </gazebo>

File: components/urdf/wam/hand.urdf.xacro (robot description, xacro)
@@ -1,29 +1,29 @@
 <robot xmlns:xacro="http://www.ros.org/wiki/xacro">
-    <xacro:include filename="$(find waterloo_steel_description)/urdf/wam/common.urdf.xacro"/>
+    <xacro:include filename="$(find uwarl-mujoco-summit-wam-sim)/components/urdf/wam/common.urdf.xacro"/>
     <xacro:property name="b" value="1.1"/>
     <!-- High-leveel hand macro -->
     <xacro:macro name="bhand" params="parent_link prefix xyz rpy">
         <xacro:bhand_palm parent_link="${parent_link}" prefix="${prefix}" xyz="${xyz}" rpy="${rpy}"/>
-        <xacro:bhand_finger_1 prefix="${prefix}"/>
-        <xacro:bhand_finger_2 prefix="${prefix}"/>
-        <xacro:bhand_finger_3 prefix="${prefix}"/>
+        <xacro:bhand_f1 prefix="${prefix}"/>
+        <xacro:bhand_f2 prefix="${prefix}"/>
+        <xacro:bhand_f3 prefix="${prefix}"/>
     </xacro:macro>
     <!-- Fingers -->
-    <xacro:macro name="bhand_finger_1" params="prefix">
-        <xacro:bhand_finger_prox prefix="${prefix}/finger_1" parent_link="${prefix}/bhand_palm_link" xyz="-0.025 0.0 0.0415" rpy="0 0 -${PI/2}" axis="0 0 -1"/>
-        <xacro:bhand_finger_med prefix="${prefix}/finger_1" parent_link="${prefix}/finger_1/prox_link" xyz="0.05 0.0 0.03390" rpy="${PI/2} 0 0"/>
-        <xacro:bhand_finger_dist prefix="${prefix}/finger_1"/>
-        <xacro:bhand_finger_tip prefix="${prefix}/finger_1"/>
-    </xacro:macro>
-    <xacro:macro name="bhand_finger_2" params="prefix">
-        <xacro:bhand_finger_prox prefix="${prefix}/finger_2" parent_link="${prefix}/bhand_palm_link" xyz="0.025 0.0 0.0415" rpy="0 0 -${PI/2}" axis="0 0 1"/>
-        <xacro:bhand_finger_med prefix="${prefix}/finger_2" parent_link="${prefix}/finger_2/prox_link" xyz="0.05 0.0 0.03390" rpy="${PI/2} 0 0"/>
-        <xacro:bhand_finger_dist prefix="${prefix}/finger_2"/>
-        <xacro:bhand_finger_tip prefix="${prefix}/finger_2"/>
-    </xacro:macro>
-    <xacro:macro name="bhand_finger_3" params="prefix">
-        <xacro:bhand_finger_med prefix="${prefix}/finger_3" parent_link="${prefix}/bhand_palm_link" xyz="0 0.05 0.0754" rpy="${PI/2} 0 ${PI/2}"/>
-        <xacro:bhand_finger_dist prefix="${prefix}/finger_3"/>
-        <xacro:bhand_finger_tip prefix="${prefix}/finger_3"/>
+    <xacro:macro name="bhand_f1" params="prefix">
+        <xacro:bhand_finger_prox prefix="${prefix}/f1" parent_link="${prefix}/bhand_palm_link" xyz="-0.025 0.0 0.0415" rpy="0 0 -${PI/2}" axis="0 0 -1"/>
+        <xacro:bhand_finger_med prefix="${prefix}/f1" parent_link="${prefix}/f1/prox_link" xyz="0.05 0.0 0.03390" rpy="${PI/2} 0 0"/>
+        <xacro:bhand_finger_dist prefix="${prefix}/f1"/>
+        <xacro:bhand_finger_tip prefix="${prefix}/f1"/>
+    </xacro:macro>
+    <xacro:macro name="bhand_f2" params="prefix">
+        <xacro:bhand_finger_prox prefix="${prefix}/f2" parent_link="${prefix}/bhand_palm_link" xyz="0.025 0.0 0.0415" rpy="0 0 -${PI/2}" axis="0 0 1"/>
+        <xacro:bhand_finger_med prefix="${prefix}/f2" parent_link="${prefix}/f2/prox_link" xyz="0.05 0.0 0.03390" rpy="${PI/2} 0 0"/>
+        <xacro:bhand_finger_dist prefix="${prefix}/f2"/>
+        <xacro:bhand_finger_tip prefix="${prefix}/f2"/>
+    </xacro:macro>
+    <xacro:macro name="bhand_f3" params="prefix">
+        <xacro:bhand_finger_med prefix="${prefix}/f3" parent_link="${prefix}/bhand_palm_link" xyz="0 0.05 0.0754" rpy="${PI/2} 0 ${PI/2}"/>
+        <xacro:bhand_finger_dist prefix="${prefix}/f3"/>
+        <xacro:bhand_finger_tip prefix="${prefix}/f3"/>
     </xacro:macro>
     <xacro:macro name="gz_hand_link" params="collide">
@@ -106,5 +106,5 @@
     </xacro:macro>
     <xacro:macro name="bhand_finger_prox" params="prefix parent_link xyz rpy axis">
-        <joint name="${prefix}/prox_joint" type="revolute">
+        <joint name="${prefix}/prox" type="revolute">
             <parent link="${parent_link}"/>
             <child link="${prefix}/prox_link"/>
@@ -114,5 +114,5 @@
             <dynamics damping="${0.1*b}" friction="0"/>
         </joint>
-        <gazebo reference="${prefix}/prox_joint">
+        <gazebo reference="${prefix}/prox">
             <xacro:gz_joint/>
         </gazebo>
@@ -147,5 +147,5 @@
     </xacro:macro>
     <xacro:macro name="bhand_finger_med" params="prefix parent_link xyz rpy">
-        <joint name="${prefix}/med_joint" type="revolute">
+        <joint name="${prefix}/med" type="revolute">
             <parent link="${parent_link}"/>
             <child link="${prefix}/med_link"/>
@@ -155,5 +155,5 @@
             <dynamics damping="${0.1*b}" friction="0"/>
         </joint>
-        <gazebo reference="${prefix}/med_joint">
+        <gazebo reference="${prefix}/med">
             <xacro:gz_joint/>
         </gazebo>
@@ -186,5 +186,5 @@
     </xacro:macro>
     <xacro:macro name="bhand_finger_dist" params="prefix">
-        <joint name="${prefix}/dist_joint" type="revolute">
+        <joint name="${prefix}/dist" type="revolute">
             <parent link="${prefix}/med_link"/>
             <child link="${prefix}/dist_link"/>
@@ -194,5 +194,5 @@
             <dynamics damping="${0.1*b}" friction="0"/>
         </joint>
-        <gazebo reference="${prefix}/dist_joint">
+        <gazebo reference="${prefix}/dist">
             <xacro:gz_joint/>
         </gazebo>

File: components/urdf/wam/wam_top.urdf.xacro (robot description, xacro)
@@ -3,13 +3,13 @@
     xmlns:controller="http://playerstage.sourceforge.net/gazebo/xmlschema/#controller">
     <!-- Some macros used by the WAM urdf -->
-    <xacro:include filename="$(find waterloo_steel_description)/urdf/wam/common.urdf.xacro"/>
+    <xacro:include filename="$(find uwarl-mujoco-summit-wam-sim)/components/urdf/wam/common.urdf.xacro"/>
     <!-- Definition of a single WAM arm -->
-    <xacro:include filename="$(find waterloo_steel_description)/urdf/wam/arm.urdf.xacro"/>
+    <xacro:include filename="$(find uwarl-mujoco-summit-wam-sim)/components/urdf/wam/arm.urdf.xacro"/>
     <!-- Definition of all the different parts of a WAM arm -->
-    <xacro:include filename="$(find waterloo_steel_description)/urdf/wam/components_V1.urdf.xacro"/>
+    <xacro:include filename="$(find uwarl-mujoco-summit-wam-sim)/components/urdf/wam/components_V1.urdf.xacro"/>
     <!-- Definitions for the barrett hand -->
-    <xacro:include filename="$(find waterloo_steel_description)/urdf/wam/hand.urdf.xacro"/>
+    <xacro:include filename="$(find uwarl-mujoco-summit-wam-sim)/components/urdf/wam/hand.urdf.xacro"/>
     <!-- Definitions for the barrett ball -->
-    <xacro:include filename="$(find waterloo_steel_description)/urdf/wam/ball.urdf.xacro"/>
+    <xacro:include filename="$(find uwarl-mujoco-summit-wam-sim)/components/urdf/wam/ball.urdf.xacro"/>
     <!-- Materials -->
     <material name="WAMGrey">
