Commit message: - Further reduced speed, since the fingers were still moving faster than what is observed from the actual hand.

File: components/urdf/wam/hand_V2.urdf.xacro (robot description, xacro)
@@ -76,5 +76,5 @@
             <child link="${prefix}/bhand_palm_surface_link"/>
             <origin xyz="0 0 0.08" rpy="0 0 0"/>
-            <limit effort="5" lower="0" upper="${PI}" velocity="0.5"/>
+            <limit effort="5" lower="0" upper="${PI}" velocity="0.2"/>
             <dynamics damping="${0.1*b}" friction="0"/>
         </joint>
@@ -92,5 +92,5 @@
             <child link="${prefix}/bhand_grasp_link"/>
             <origin xyz="0 0 0.12" rpy="0 0 0"/>
-            <limit effort="5" lower="0" upper="${PI}" velocity="0.5"/>
+            <limit effort="5" lower="0" upper="${PI}" velocity="0.2"/>
             <dynamics damping="${0.1*b}" friction="0"/>
         </joint>
@@ -111,5 +111,5 @@
             <origin xyz="${xyz}" rpy="${rpy}"/>
             <axis xyz="${axis}"/>
-            <limit effort="5" lower="0" upper="${PI}" velocity="0.5"/>
+            <limit effort="5" lower="0" upper="${PI}" velocity="0.2"/>
             <dynamics damping="${0.1*b}" friction="0"/>
         </joint>
@@ -152,5 +152,5 @@
             <origin xyz="${xyz}" rpy="${rpy}"/>
             <axis xyz="0 0 1"/>
-            <limit effort="5" lower="0" upper="${140/180*PI}" velocity="0.5"/>
+            <limit effort="5" lower="0" upper="${140/180*PI}" velocity="0.2"/>
             <dynamics damping="${0.1*b}" friction="0"/>
         </joint>
@@ -191,5 +191,5 @@
             <origin xyz="0.06994 0.003 0.0" rpy="0 0 ${PI/4}"/>
             <axis xyz="0 0 1"/>
-            <limit effort="5" lower="0" upper="${48/180*PI}" velocity="0.5"/>
+            <limit effort="5" lower="0" upper="${48/180*PI}" velocity="0.2"/>
             <dynamics damping="${0.1*b}" friction="0"/>
         </joint>
