Commit message: - Fetch xacro-file bodies and joints have been re-named to be the same as the mujoco model.

File: components/robots/fetch_mujoco.urdf.xacro (robot description, xacro)
@@ -10,8 +10,10 @@
     <xacro:include filename="$(find uwarl-mujoco-summit-wam-sim)/components/urdf/fetch/fetch_gazebo.xacro"/>
     <!-- Construct Fetch Base -->
-    <xacro:base prefix="fetch"/>
-    <xacro:body prefix="fetch"/>
-    <xacro:head prefix="fetch"/>
-    <xacro:arm prefix="fetch"/>
-    <xacro:gripper prefix="fetch"/>
+    <!-- https://answers.ros.org/question/282902/pass-parameters-to-xacro-from-launch-file-or-otherwise/ -->
+    <xacro:arg name="prefix" default="fetch" />
+    <xacro:base prefix="$(arg prefix)"/>
+    <xacro:body prefix="$(arg prefix)"/>
+    <xacro:head prefix="$(arg prefix)"/>
+    <xacro:arm prefix="$(arg prefix)"/>
+    <xacro:gripper prefix="$(arg prefix)"/>
 </robot>

File: components/urdf/fetch/arm.xacro (robot description, xacro)
@@ -3,5 +3,5 @@
     <!-- Mesh from https://www.blendswap.com/blends/view/74733-->
     <xacro:macro name="arm" params="prefix">
-        <link name="${prefix}_shoulder_pan_link">
+        <link name="${prefix}/shoulder_pan_link">
             <inertial>
                 <origin rpy="0 0 0" xyz="0.0927 -0.0056 0.0564" />
@@ -25,23 +25,23 @@
             </collision>
         </link>
-        <joint name="${prefix}_shoulder_pan_joint" type="revolute">
+        <joint name="${prefix}/shoulder_pan" type="revolute">
             <origin rpy="0 0 0" xyz="0.119525 0 0.34858" />
-            <parent link="${prefix}_torso_lift_link" />
-            <child link="${prefix}_shoulder_pan_link" />
+            <parent link="${prefix}/torso_lift_link" />
+            <child link="${prefix}/shoulder_pan_link" />
             <axis xyz="0 0 1" />
             <dynamics damping="1.0" />
             <limit effort="33.82" lower="-1.6056" upper="1.6056" velocity="1.256" />
         </joint>
-        <transmission name="${prefix}_shoulder_pan_joint_tran">
-            <type>transmission_interface/SimpleTransmission</type>
-            <joint name="${prefix}_shoulder_pan_joint">
-                <hardwareInterface>EffortJointInterface</hardwareInterface>
-            </joint>
-            <actuator name="${prefix}_shoulder_pan_joint_motor">
-                <hardwareInterface>EffortJointInterface</hardwareInterface>
-                <mechanicalReduction>1</mechanicalReduction>
-            </actuator>
-        </transmission>
-        <link name="${prefix}_shoulder_lift_link">
+        <transmission name="${prefix}shoulder_pan_joint_tran">
+            <type>transmission_interface/SimpleTransmission</type>
+            <joint name="${prefix}/shoulder_pan">
+                <hardwareInterface>hardware_interface/EffortJointInterface</hardwareInterface>
+            </joint>
+            <actuator name="${prefix}shoulder_pan_joint_motor">
+                <!-- <hardwareInterface>EffortJointInterface</hardwareInterface> -->
+                <mechanicalReduction>1</mechanicalReduction>
+            </actuator>
+        </transmission>
+        <link name="${prefix}/shoulder_lift_link">
             <inertial>
                 <origin rpy="0 0 0" xyz="0.1432 0.0072 -0.0001" />
@@ -65,23 +65,23 @@
             </collision>
         </link>
-        <joint name="${prefix}_shoulder_lift_joint" type="revolute">
+        <joint name="${prefix}/shoulder_lift" type="revolute">
             <origin rpy="0 0 0" xyz="0.117 0 0.0599999999999999" />
-            <parent link="${prefix}_shoulder_pan_link" />
-            <child link="${prefix}_shoulder_lift_link" />
+            <parent link="${prefix}/shoulder_pan_link" />
+            <child link="${prefix}/shoulder_lift_link" />
             <axis xyz="0 1 0" />
             <dynamics damping="1.0" />
             <limit effort="131.76" lower="-1.221" upper="1.518" velocity="1.454" />
         </joint>
-        <transmission name="${prefix}_shoulder_lift_joint_tran">
-            <type>transmission_interface/SimpleTransmission</type>
-            <joint name="${prefix}_shoulder_lift_joint">
-                <hardwareInterface>EffortJointInterface</hardwareInterface>
-            </joint>
-            <actuator name="${prefix}_shoulder_lift_joint_motor">
-                <hardwareInterface>EffortJointInterface</hardwareInterface>
-                <mechanicalReduction>1</mechanicalReduction>
-            </actuator>
-        </transmission>
-        <link name="${prefix}_upperarm_roll_link">
+        <transmission name="${prefix}shoulder_lift_joint_tran">
+            <type>transmission_interface/SimpleTransmission</type>
+            <joint name="${prefix}/shoulder_lift">
+                <hardwareInterface>hardware_interface/EffortJointInterface</hardwareInterface>
+            </joint>
+            <actuator name="${prefix}shoulder_lift_joint_motor">
+                <!-- <hardwareInterface>EffortJointInterface</hardwareInterface> -->
+                <mechanicalReduction>1</mechanicalReduction>
+            </actuator>
+        </transmission>
+        <link name="${prefix}/upper_arm_roll_link">
             <inertial>
                 <origin rpy="0 0 0" xyz="0.1165 0.0014 0.0000" />
@@ -105,23 +105,23 @@
             </collision>
         </link>
-        <joint name="${prefix}_upperarm_roll_joint" type="continuous">
+        <joint name="${prefix}/upper_arm_roll" type="continuous">
             <origin rpy="0 0 0" xyz="0.219 0 0" />
-            <parent link="${prefix}_shoulder_lift_link" />
-            <child link="${prefix}_upperarm_roll_link" />
+            <parent link="${prefix}/shoulder_lift_link" />
+            <child link="${prefix}/upper_arm_roll_link" />
             <axis xyz="1 0 0" />
             <dynamics damping="5.0" />
             <limit effort="76.94" velocity="1.571" />
         </joint>
-        <transmission name="${prefix}_upperarm_roll_joint_tran">
-            <type>transmission_interface/SimpleTransmission</type>
-            <joint name="${prefix}_upperarm_roll_joint">
-                <hardwareInterface>EffortJointInterface</hardwareInterface>
-            </joint>
-            <actuator name="${prefix}_upperarm_roll_joint_motor">
-                <hardwareInterface>EffortJointInterface</hardwareInterface>
-                <mechanicalReduction>1</mechanicalReduction>
-            </actuator>
-        </transmission>
-        <link name="${prefix}_elbow_flex_link">
+        <transmission name="${prefix}/upper_arm_roll_joint_tran">
+            <type>transmission_interface/SimpleTransmission</type>
+            <joint name="${prefix}/upper_arm_roll">
+                <hardwareInterface>hardware_interface/EffortJointInterface</hardwareInterface>
+            </joint>
+            <actuator name="${prefix}/upper_arm_roll_joint_motor">
+                <!-- <hardwareInterface>EffortJointInterface</hardwareInterface> -->
+                <mechanicalReduction>1</mechanicalReduction>
+            </actuator>
+        </transmission>
+        <link name="${prefix}/elbow_flex_link">
             <inertial>
                 <origin rpy="0 0 0" xyz="0.1279 0.0073 0.0000" />
@@ -145,23 +145,23 @@
             </collision>
         </link>
-        <joint name="${prefix}_elbow_flex_joint" type="revolute">
+        <joint name="${prefix}/elbow_flex" type="revolute">
             <origin rpy="0 0 0" xyz="0.133 0 0" />
-            <parent link="${prefix}_upperarm_roll_link" />
-            <child link="${prefix}_elbow_flex_link" />
+            <parent link="${prefix}/upper_arm_roll_link" />
+            <child link="${prefix}/elbow_flex_link" />
             <axis xyz="0 1 0" />
             <dynamics damping="1.0" />
             <limit effort="66.18" lower="-2.251" upper="2.251" velocity="1.521" />
         </joint>
-        <transmission name="${prefix}_elbow_flex_joint_tran">
-            <type>transmission_interface/SimpleTransmission</type>
-            <joint name="${prefix}_elbow_flex_joint">
-                <hardwareInterface>EffortJointInterface</hardwareInterface>
-            </joint>
-            <actuator name="${prefix}_elbow_flex_joint_motor">
-                <hardwareInterface>EffortJointInterface</hardwareInterface>
-                <mechanicalReduction>1</mechanicalReduction>
-            </actuator>
-        </transmission>
-        <link name="${prefix}_forearm_roll_link">
+        <transmission name="${prefix}/elbow_flex_joint_tran">
+            <type>transmission_interface/SimpleTransmission</type>
+            <joint name="${prefix}/elbow_flex">
+                <hardwareInterface>hardware_interface/EffortJointInterface</hardwareInterface>
+            </joint>
+            <actuator name="${prefix}/elbow_flex_joint_motor">
+                <!-- <hardwareInterface>EffortJointInterface</hardwareInterface> -->
+                <mechanicalReduction>1</mechanicalReduction>
+            </actuator>
+        </transmission>
+        <link name="${prefix}/fore_arm_roll_link">
             <inertial>
                 <origin rpy="0 0 0" xyz="0.1097 -0.0266 0.0000" />
@@ -185,23 +185,23 @@
             </collision>
         </link>
-        <joint name="${prefix}_forearm_roll_joint" type="continuous">
+        <joint name="${prefix}/fore_arm_roll" type="continuous">
             <origin rpy="0 0 0" xyz="0.197 0 0" />
-            <parent link="${prefix}_elbow_flex_link" />
-            <child link="${prefix}_forearm_roll_link" />
+            <parent link="${prefix}/elbow_flex_link" />
+            <child link="${prefix}/fore_arm_roll_link" />
             <axis xyz="1 0 0" />
             <dynamics damping="5.0" />
             <limit effort="29.35" velocity="1.571" />
         </joint>
-        <transmission name="${prefix}_forearm_roll_joint_tran">
-            <type>transmission_interface/SimpleTransmission</type>
-            <joint name="${prefix}_forearm_roll_joint">
-                <hardwareInterface>EffortJointInterface</hardwareInterface>
-            </joint>
-            <actuator name="${prefix}_forearm_roll_joint_motor">
-                <hardwareInterface>EffortJointInterface</hardwareInterface>
-                <mechanicalReduction>1</mechanicalReduction>
-            </actuator>
-        </transmission>
-        <link name="${prefix}_wrist_flex_link">
+        <transmission name="${prefix}/fore_arm_roll_joint_tran">
+            <type>transmission_interface/SimpleTransmission</type>
+            <joint name="${prefix}/fore_arm_roll">
+                <hardwareInterface>hardware_interface/EffortJointInterface</hardwareInterface>
+            </joint>
+            <actuator name="${prefix}/fore_arm_roll_joint_motor">
+                <!-- <hardwareInterface>EffortJointInterface</hardwareInterface> -->
+                <mechanicalReduction>1</mechanicalReduction>
+            </actuator>
+        </transmission>
+        <link name="${prefix}/wrist_flex_link">
             <inertial>
                 <origin rpy="0 0 0" xyz="0.0882 0.0009 -0.0001" />
@@ -225,23 +225,23 @@
             </collision>
         </link>
-        <joint name="${prefix}_wrist_flex_joint" type="revolute">
+        <joint name="${prefix}/wrist_flex" type="revolute">
             <origin rpy="0 0 0" xyz="0.1245 0 0" />
-            <parent link="${prefix}_forearm_roll_link" />
-            <child link="${prefix}_wrist_flex_link" />
+            <parent link="${prefix}/fore_arm_roll_link" />
+            <child link="${prefix}/wrist_flex_link" />
             <axis xyz="0 1 0" />
             <dynamics damping="1.0" />
             <limit effort="25.7" lower="-2.16" upper="2.16" velocity="2.268" />
         </joint>
-        <transmission name="${prefix}_wrist_flex_joint_tran">
-            <type>transmission_interface/SimpleTransmission</type>
-            <joint name="${prefix}_wrist_flex_joint">
-                <hardwareInterface>EffortJointInterface</hardwareInterface>
-            </joint>
-            <actuator name="${prefix}_wrist_flex_joint_motor">
-                <hardwareInterface>EffortJointInterface</hardwareInterface>
-                <mechanicalReduction>1</mechanicalReduction>
-            </actuator>
-        </transmission>
-        <link name="${prefix}_wrist_roll_link">
+        <transmission name="${prefix}/wrist_flex_joint_tran">
+            <type>transmission_interface/SimpleTransmission</type>
+            <joint name="${prefix}/wrist_flex">
+                <hardwareInterface>hardware_interface/EffortJointInterface</hardwareInterface>
+            </joint>
+            <actuator name="${prefix}/wrist_flex_joint_motor">
+                <!-- <hardwareInterface>EffortJointInterface</hardwareInterface> -->
+                <mechanicalReduction>1</mechanicalReduction>
+            </actuator>
+        </transmission>
+        <link name="${prefix}/wrist_roll_link">
             <inertial>
                 <origin rpy="0 0 0" xyz="0.0095 0.0004 -0.0002" />
@@ -265,19 +265,19 @@
             </collision>
         </link>
-        <joint name="${prefix}_wrist_roll_joint" type="continuous">
+        <joint name="${prefix}/wrist_roll" type="continuous">
             <origin rpy="0 0 0" xyz="0.1385 0 0" />
-            <parent link="${prefix}_wrist_flex_link" />
-            <child link="${prefix}_wrist_roll_link" />
+            <parent link="${prefix}/wrist_flex_link" />
+            <child link="${prefix}/wrist_roll_link" />
             <axis xyz="1 0 0" />
             <limit effort="7.36" velocity="2.268" />
             <dynamics damping="5.0" />
         </joint>
-        <transmission name="${prefix}_wrist_roll_joint_tran">
-            <type>transmission_interface/SimpleTransmission</type>
-            <joint name="${prefix}_wrist_roll_joint">
-                <hardwareInterface>EffortJointInterface</hardwareInterface>
-            </joint>
-            <actuator name="${prefix}_wrist_roll_joint_motor">
-                <hardwareInterface>EffortJointInterface</hardwareInterface>
+        <transmission name="${prefix}/wrist_roll_joint_tran">
+            <type>transmission_interface/SimpleTransmission</type>
+            <joint name="${prefix}/wrist_roll">
+                <hardwareInterface>hardware_interface/EffortJointInterface</hardwareInterface>
+            </joint>
+            <actuator name="${prefix}/wrist_roll_joint_motor">
+                <!-- <hardwareInterface>EffortJointInterface</hardwareInterface> -->
                 <mechanicalReduction>1</mechanicalReduction>
             </actuator>

File: components/urdf/fetch/base.xacro (robot description, xacro)
@@ -3,11 +3,11 @@
     <!-- Mesh from https://www.blendswap.com/blends/view/74733-->
     <xacro:macro name="base" params="prefix">
-        <link name="${prefix}_base_footprint"/>
-        <joint name="${prefix}_base_footprint_joint" type="fixed">
+        <link name="${prefix}/base_footprint"/>
+        <joint name="${prefix}/base_footprint_joint" type="fixed">
             <origin rpy="0 0 0" xyz="0 0 0" />
-            <parent link="${prefix}_base_footprint" />
-            <child link="${prefix}_base_link" />
+            <parent link="${prefix}/base_footprint" />
+            <child link="${prefix}/base_link" />
         </joint>
-        <link name="${prefix}_base_link">
+        <link name="${prefix}/base_link">
             <inertial>
                 <origin rpy="0 0 0" xyz="-0.0036 0.0 0.0014" />
@@ -31,5 +31,5 @@
             </collision>
         </link>
-        <link name="${prefix}_r_wheel_link">
+        <link name="${prefix}/whl/R_link">
             <inertial>
                 <origin rpy="0 0 0" xyz="0 0 0" />
@@ -53,12 +53,12 @@
             </collision>
         </link>
-        <joint name="${prefix}_r_wheel_joint" type="continuous">
+        <joint name="${prefix}/R_whl" type="continuous">
             <origin rpy="-6.123E-17 0 0" xyz="0.0012914 ${-1*wheel_center_dist_y} 0.055325" />
-            <parent link="${prefix}_base_link" />
-            <child link="${prefix}_r_wheel_link" />
+            <parent link="${prefix}/base_link" />
+            <child link="${prefix}/whl/R_link" />
             <axis xyz="0 1 0" />
             <limit effort="8.85" velocity="17.4" />
         </joint>
-        <link name="${prefix}_l_wheel_link">
+        <link name="${prefix}/whl/L_link">
             <inertial>
                 <origin rpy="0 0 0" xyz="0 0 0" />
@@ -82,8 +82,8 @@
             </collision>
         </link>
-        <joint name="${prefix}_l_wheel_joint" type="continuous">
+        <joint name="${prefix}/L_whl" type="continuous">
             <origin rpy="-6.123E-17 0 0" xyz="0.0012914 ${wheel_center_dist_y} 0.055325" />
-            <parent link="${prefix}_base_link" />
-            <child link="${prefix}_l_wheel_link" />
+            <parent link="${prefix}/base_link" />
+            <child link="${prefix}/whl/L_link" />
             <axis xyz="0 1 0" />
             <limit effort="8.85" velocity="17.4" />
