Commit message: - Fetch xacro-file bodies and joints have been re-named to be the same as the mujoco model.

File: components/urdf/fetch/body.xacro (robot description, xacro)
@@ -3,5 +3,5 @@
     <!-- Mesh from https://www.blendswap.com/blends/view/74733-->
     <xacro:macro name="body" params="prefix">
-        <link name="${prefix}_torso_lift_link">
+        <link name="${prefix}/torso_lift_link">
             <inertial>
                 <origin rpy="0 0 0" xyz="-0.0013 -0.0009 0.2935" />
@@ -25,23 +25,23 @@
             </collision>
         </link>
-        <joint name="${prefix}_torso_lift_joint" type="prismatic">
+        <joint name="${prefix}/torso_lift" type="prismatic">
             <origin rpy="-6.123E-17 0 0" xyz="-0.086875 0 0.37743" />
-            <parent link="${prefix}_base_link" />
-            <child link="${prefix}_torso_lift_link" />
+            <parent link="${prefix}/base_link" />
+            <child link="${prefix}/torso_lift_link" />
             <axis xyz="0 0 1" />
             <limit effort="450.0" lower="0" upper="0.38615" velocity="0.1" />
             <dynamics damping="100.0" />
         </joint>
-        <transmission name="${prefix}_torso_lift_joint_tran">
+        <transmission name="${prefix}/torso_lift_joint_tran">
             <type>transmission_interface/SimpleTransmission</type>
-            <joint name="${prefix}_torso_lift_joint">
-                <hardwareInterface>EffortJointInterface</hardwareInterface>
+            <joint name="${prefix}/torso_lift">
+                <hardwareInterface>hardware_interface/EffortJointInterface</hardwareInterface>
             </joint>
-            <actuator name="${prefix}_torso_lift_joint_motor">
-                <hardwareInterface>EffortJointInterface</hardwareInterface>
+            <actuator name="${prefix}/torso_lift_joint_motor">
+                <!-- <hardwareInterface>EffortJointInterface</hardwareInterface> -->
                 <mechanicalReduction>1</mechanicalReduction>
             </actuator>
         </transmission>
-        <link name="${prefix}_bellows_link">
+        <link name="${prefix}/bellows_link">
             <inertial>
                 <origin rpy="0 0 0" xyz="0.0191320000286228 -1.67219873481315E-16 -0.134861625443387" />
@@ -65,22 +65,10 @@
             </collision>
         </link>
-        <joint name="${prefix}_bellows_joint" type="prismatic">
+        <joint name="${prefix}/bellows_joint" type="fixed">
             <origin rpy="0 0 0" xyz="0 0 0" />
-            <parent link="${prefix}_torso_lift_link" />
-            <child link="${prefix}_bellows_link" />
-            <axis xyz="0 0 1" />
-            <limit effort="5.0" lower="0" upper="0.4" velocity="0.1" />
+            <parent link="${prefix}/torso_lift_link" />
+            <child link="${prefix}/bellows_link" />
         </joint>
-        <transmission name="${prefix}_bellows_joint_tran">
-            <type>transmission_interface/SimpleTransmission</type>
-            <joint name="${prefix}_bellows_joint">
-                <hardwareInterface>EffortJointInterface</hardwareInterface>
-            </joint>
-            <actuator name="${prefix}_bellows_joint_motor">
-                <hardwareInterface>EffortJointInterface</hardwareInterface>
-                <mechanicalReduction>1</mechanicalReduction>
-            </actuator>
-        </transmission>
-        <link name="${prefix}_bellows_link2">
+        <link name="${prefix}/bellows_2_link">
             <inertial>
                 <origin rpy="0 0 0" xyz="0.0191320000286228 -1.67219873481315E-16 -0.134861625443387" />
@@ -104,12 +92,10 @@
             </collision>
         </link>
-        <joint name="${prefix}_bellows_joint2" type="prismatic">
+        <joint name="${prefix}/bellows_2_joint" type="fixed">
             <origin rpy="0 0 3.1415927" xyz="-0.14 0 0" />
-            <parent link="${prefix}_torso_lift_link" />
-            <child link="${prefix}_bellows_link2" />
-            <axis xyz="0 0 1" />
-            <limit effort="5.0" lower="0" upper="0.4" velocity="0.1" />
+            <parent link="${prefix}/torso_lift_link" />
+            <child link="${prefix}/bellows_2_link" />
         </joint>
-        <link name="${prefix}_estop_link">
+        <link name="${prefix}/e_stop_link">
             <inertial>
                 <origin rpy="0 0 0" xyz="0.002434512737072 -0.00330608315239905 0.00665139196650039" />
@@ -133,11 +119,11 @@
             </collision>
         </link>
-        <joint name="${prefix}_estop_joint" type="fixed">
+        <joint name="${prefix}/e_stop_joint" type="fixed">
             <origin rpy="1.5708 0 0" xyz="-0.12465 0.23892 0.31127" />
-            <parent link="${prefix}_base_link" />
-            <child link="${prefix}_estop_link" />
+            <parent link="${prefix}/base_link" />
+            <child link="${prefix}/e_stop_link" />
         <axis xyz="0 0 0" />
         </joint>
-        <link name="${prefix}_laser_link">
+        <link name="${prefix}/laser_link">
             <inertial>
                 <origin rpy="0 0 0" xyz="-0.0306228970175641 0.0007091682908278 0.0551974119471302" />
@@ -161,11 +147,11 @@
             </collision>
         </link>
-        <joint name="${prefix}_laser_joint" type="fixed">
+        <joint name="${prefix}/laser_joint" type="fixed">
             <origin rpy="3.14159265359 0 0" xyz="0.235 0 0.2878" />
-            <parent link="${prefix}_base_link" />
-            <child link="${prefix}_laser_link" />
+            <parent link="${prefix}/base_link" />
+            <child link="${prefix}/laser_link" />
             <axis xyz="0 0 0" />
         </joint>
-        <link name="${prefix}_torso_fixed_link">
+        <link name="${prefix}/torso_fixed_link">
             <inertial>
                 <origin rpy="0 0 0" xyz="-0.0722 0.0057 0.2656" />
@@ -189,8 +175,8 @@
             </collision>
         </link>
-        <joint name="${prefix}_torso_fixed_joint" type="fixed">
+        <joint name="${prefix}/torso_fixed_joint" type="fixed">
             <origin rpy="-6.12303176911189E-17 0 0" xyz="-0.086875 0 0.377425" />
-            <parent link="${prefix}_base_link" />
-            <child link="${prefix}_torso_fixed_link" />
+            <parent link="${prefix}/base_link" />
+            <child link="${prefix}/torso_fixed_link" />
             <axis xyz="0 1 0" />
         </joint>

File: components/urdf/fetch/gripper.xacro (robot description, xacro)
@@ -3,5 +3,5 @@
     <!-- Mesh from https://www.blendswap.com/blends/view/74733-->
     <xacro:macro name="gripper" params="prefix">
-        <link name="${prefix}_gripper_link">
+        <link name="${prefix}/gripper_link">
             <inertial>
                 <origin rpy="0 0 0" xyz="-0.0900 -0.0001 -0.0017" />
@@ -22,11 +22,11 @@
             </collision>
         </link>
-        <joint name="${prefix}_gripper_axis" type="fixed">
+        <joint name="${prefix}/gripper_axis" type="fixed">
             <origin rpy="0 0 0" xyz="0.16645 0 0" />
-            <parent link="${prefix}_wrist_roll_link" />
-            <child link="${prefix}_gripper_link" />
+            <parent link="${prefix}/wrist_roll_link" />
+            <child link="${prefix}/gripper_link" />
             <axis xyz="0 1 0" />
         </joint>
-        <link name="${prefix}_r_gripper_finger_link">
+        <link name="${prefix}/right_gripper_finger_link">
             <inertial>
                 <origin rpy="0 0 0" xyz="-0.01 0 0" />
@@ -50,25 +50,27 @@
             </collision>
         </link>
-        <joint name="${prefix}_r_gripper_finger_joint" type="prismatic">
+        <joint name="${prefix}/right_gripper_finger" type="prismatic">
             <origin rpy="0 0 0" xyz="0 0.015425 0" />
-            <parent link="${prefix}_gripper_link" />
-            <child link="${prefix}_r_gripper_finger_link" />
+            <parent link="${prefix}/gripper_link" />
+            <child link="${prefix}/right_gripper_finger_link" />
             <axis xyz="0 1 0" />
             <limit effort="60" lower="0.0" upper="0.05" velocity="0.05" /><dynamics damping="100.0" />
         </joint>
-        <transmission name="${prefix}_r_gripper_finger_joint_tran">
+        <transmission name="${prefix}/right_gripper_finger_joint_tran">
             <type>transmission_interface/SimpleTransmission</type>
-            <joint name="${prefix}_r_gripper_finger_joint">
-                <hardwareInterface>EffortJointInterface</hardwareInterface>
+            <joint name="${prefix}/right_gripper_finger">
+                <hardwareInterface>hardware_interface/EffortJointInterface</hardwareInterface>
             </joint>
-            <actuator name="${prefix}_r_gripper_finger_joint_motor">
-                <hardwareInterface>EffortJointInterface</hardwareInterface>
+            <actuator name="${prefix}/right_gripper_finger_joint_motor">
+                <!-- <hardwareInterface>EffortJointInterface</hardwareInterface> -->
                 <mechanicalReduction>1</mechanicalReduction>
             </actuator>
         </transmission>
-        <link name="${prefix}_l_gripper_finger_link">
+        <link name="${prefix}/left_gripper_finger_link">
             <inertial>
                 <origin rpy="0 0 0" xyz="-0.01 0 0" />
                 <mass value="0.0798" />
+                <!-- Error: inertia must satisfy A + B >= C -->
+                <!-- https://physics.stackexchange.com/a/48273 -->
                 <inertia ixx="0.002" ixy="0" ixz="0" iyy="0" iyz="0" izz="0" />
             </inertial>
@@ -89,18 +91,18 @@
             </collision>
         </link>
-        <joint name="${prefix}_l_gripper_finger_joint" type="prismatic">
+        <joint name="${prefix}/left_gripper_finger_joint" type="prismatic">
             <origin rpy="0 0 0" xyz="0 -0.015425 0" />
-            <parent link="${prefix}_gripper_link" />
-            <child link="${prefix}_l_gripper_finger_link" />
+            <parent link="${prefix}/gripper_link" />
+            <child link="${prefix}/left_gripper_finger_link" />
             <axis xyz="0 -1 0" />
             <limit effort="60" lower="0.0" upper="0.05" velocity="0.05" /><dynamics damping="100.0" />
         </joint>
-        <transmission name="${prefix}_l_gripper_finger_joint_tran">
+        <transmission name="${prefix}/left_gripper_finger_joint_tran">
             <type>transmission_interface/SimpleTransmission</type>
-            <joint name="${prefix}_l_gripper_finger_joint">
-                <hardwareInterface>EffortJointInterface</hardwareInterface>
+            <joint name="${prefix}/left_gripper_finger">
+                <hardwareInterface>hardware_interface/EffortJointInterface</hardwareInterface>
             </joint>
-            <actuator name="${prefix}_l_gripper_finger_joint_motor">
-                <hardwareInterface>EffortJointInterface</hardwareInterface>
+            <actuator name="${prefix}/left_gripper_finger_joint_motor">
+                <!-- <hardwareInterface>EffortJointInterface</hardwareInterface> -->
                 <mechanicalReduction>1</mechanicalReduction>
             </actuator>

File: components/urdf/fetch/head.xacro (robot description, xacro)
@@ -3,5 +3,5 @@
     <!-- Mesh from https://www.blendswap.com/blends/view/74733-->
     <xacro:macro name="head" params="prefix">
-        <link name="${prefix}_head_pan_link">
+        <link name="${prefix}/head_pan_link">
             <inertial>
                 <origin rpy="0 0 0" xyz="0.0321 0.0161 0.0390" />
@@ -25,22 +25,22 @@
             </collision>
         </link>
-        <joint name="${prefix}_head_pan_joint" type="revolute">
+        <joint name="${prefix}/head_pan" type="revolute">
             <origin rpy="0 0 0" xyz="0.053125 0 0.603001417713939" />
-            <parent link="${prefix}_torso_lift_link" />
-            <child link="${prefix}_head_pan_link" />
+            <parent link="${prefix}/torso_lift_link" />
+            <child link="${prefix}/head_pan_link" />
             <axis xyz="0 0 1" />
             <limit effort="0.32" lower="-1.57" upper="1.57" velocity="1.57" />
         </joint>
-        <transmission name="${prefix}_head_pan_joint_tran">
+        <transmission name="${prefix}/head_pan_joint_tran">
             <type>transmission_interface/SimpleTransmission</type>
-            <joint name="${prefix}_head_pan_joint">
-                <hardwareInterface>EffortJointInterface</hardwareInterface>
+            <joint name="${prefix}/head_pan">
+                <hardwareInterface>hardware_interface/EffortJointInterface</hardwareInterface>
             </joint>
-            <actuator name="${prefix}_head_pan_joint_motor">
-                <hardwareInterface>EffortJointInterface</hardwareInterface>
+            <actuator name="${prefix}head_pan_joint_motor">
+                <!-- <hardwareInterface>EffortJointInterface</hardwareInterface> -->
                 <mechanicalReduction>1</mechanicalReduction>
             </actuator>
         </transmission>
-        <link name="${prefix}_head_tilt_link">
+        <link name="${prefix}/head_tilt_link">
             <inertial>
                 <origin rpy="0 0 0" xyz="0.0081 0.0025 0.0113" />
@@ -64,50 +64,50 @@
             </collision>
         </link>
-        <joint name="${prefix}_head_tilt_joint" type="revolute">
+        <joint name="${prefix}/head_tilt" type="revolute">
             <origin rpy="0 0 0" xyz="0.14253 0 0.057999" />
-            <parent link="${prefix}_head_pan_link" />
-            <child link="${prefix}_head_tilt_link" />
+            <parent link="${prefix}/head_pan_link" />
+            <child link="${prefix}/head_tilt_link" />
             <axis xyz="0 1 0" />
             <limit effort="0.68" lower="-0.76" upper="1.45" velocity="1.57" />
         </joint>
-        <transmission name="${prefix}_head_tilt_joint_tran">
+        <transmission name="${prefix}head_tilt_joint_tran">
             <type>transmission_interface/SimpleTransmission</type>
-            <joint name="${prefix}_head_tilt_joint">
-                <hardwareInterface>EffortJointInterface</hardwareInterface>
+            <joint name="${prefix}/head_tilt">
+                <hardwareInterface>hardware_interface/EffortJointInterface</hardwareInterface>
             </joint>
-            <actuator name="${prefix}_head_tilt_joint_motor">
-                <hardwareInterface>EffortJointInterface</hardwareInterface>
+            <actuator name="${prefix}head_tilt_joint_motor">
+                <!-- <hardwareInterface>EffortJointInterface</hardwareInterface> -->
                 <mechanicalReduction>1</mechanicalReduction>
             </actuator>
         </transmission>
-        <link name="${prefix}_head_camera_link" />
-        <joint name="${prefix}_head_camera_joint" type="fixed">
+        <link name="${prefix}/head_camera_link" />
+        <joint name="${prefix}/head_camera_joint" type="fixed">
             <origin rpy="0 0 0" xyz="0.055 0 0.0225" />
-            <parent link="head_tilt_link" />
-            <child link="head_camera_link" />
+            <parent link="${prefix}/head_tilt_link" />
+            <child link="${prefix}/head_camera_link" />
         </joint>
-        <link name="${prefix}_head_camera_rgb_frame" />
-        <joint name="${prefix}_head_camera_rgb_joint" type="fixed">
+        <link name="${prefix}/head_camera_rgb_frame" />
+        <joint name="${prefix}/head_camera_rgb_joint" type="fixed">
             <origin rpy="0 0 0" xyz="0 0.02 0" />
-            <parent link="${prefix}_head_camera_link" />
-            <child link="${prefix}_head_camera_rgb_frame" />
+            <parent link="${prefix}/head_camera_link" />
+            <child link="${prefix}/head_camera_rgb_frame" />
         </joint>
-        <link name="${prefix}_head_camera_rgb_optical_frame" />
-        <joint name="${prefix}_head_camera_rgb_optical_joint" type="fixed">
+        <link name="${prefix}/head_camera_rgb_optical_frame" />
+        <joint name="${prefix}/head_camera_rgb_optical_joint" type="fixed">
             <origin rpy="-1.57079632679 0 -1.57079632679" xyz="0 0 0" />
-            <parent link="${prefix}_head_camera_rgb_frame" />
-            <child link="${prefix}_head_camera_rgb_optical_frame" />
+            <parent link="${prefix}/head_camera_rgb_frame" />
+            <child link="${prefix}/head_camera_rgb_optical_frame" />
         </joint>
-        <link name="${prefix}_head_camera_depth_frame" />
-        <joint name="${prefix}_head_camera_depth_joint" type="fixed">
+        <link name="${prefix}/head_camera_depth_frame" />
+        <joint name="${prefix}/head_camera_depth_joint" type="fixed">
             <origin rpy="0 0 0" xyz="0 0.045 0" />
-            <parent link="${prefix}_head_camera_link" />
-            <child link="${prefix}_head_camera_depth_frame" />
+            <parent link="${prefix}/head_camera_link" />
+            <child link="${prefix}/head_camera_depth_frame" />
         </joint>
-        <link name="${prefix}_head_camera_depth_optical_frame" />
-        <joint name="${prefix}_head_camera_depth_optical_joint" type="fixed">
+        <link name="${prefix}/head_camera_depth_optical_frame" />
+        <joint name="${prefix}/head_camera_depth_optical_joint" type="fixed">
             <origin rpy="-1.57079632679 0 -1.57079632679" xyz="0 0 0" />
-            <parent link="${prefix}_head_camera_depth_frame" />
-            <child link="${prefix}_head_camera_depth_optical_frame" />
+            <parent link="${prefix}/head_camera_depth_frame" />
+            <child link="${prefix}/head_camera_depth_optical_frame" />
         </joint>
     </xacro:macro>
