Commit message: - Temporarily diabled the camera-view, - Added gear-ratios and position constraints on the joints of the fetch. This seems to have allowed the Fetch arm to behave well; yet the simulation still continues to reset periodically.

File: components/urdf/fetch/gripper.xacro (robot description, xacro)
@@ -91,5 +91,5 @@
             </collision>
         </link>
-        <joint name="${prefix}_hand/left_gripper_finger_joint" type="prismatic">
+        <joint name="${prefix}_hand/left_gripper_finger" type="prismatic">
             <origin rpy="0 0 0" xyz="0 -0.015425 0" />
             <parent link="${prefix}_hand/gripper_link" />
